File: kicad/4-in-power-improved.kicad_pcb (KiCad board)
At the start: 2 copper layers, 84.1 x 61.7 mm, 189 parts, among them J1 USB_C_Receptacle_USB2.0_16P, J2 Bus_PCI_Express_x1, J3 Conn_01x02, Q1 FMMT493, Q2 AO3400A, Q3 AO3400A, U1 XC6206P332MR, U10 BQ25672RQMR, U11 TPS54331DR, U12 6.8uH, U13 TPS54331DR, U14 6.8uH, U15 6.8uH, U16 SX1308, U2 2P SMD 2.54P Jumper, U3 W25Q128JVP, U4 2P SMD 2.54P Jumper, U5 MCP25625T-E/ML, U6 RP2040, U7 S5B-XH-A(LF)(SN), U8 XT30PW-M, U9 BQ7694202PFBR, X1 ABM8-272-T3, Y1 X322516MLB4SI

Commit message: Charger IC footprint routed RP2040 routed BMS routed xt30s and balancers router
Parts:
- removed C27: 220nF, PCM_JLCPCB:C_0805
- added C76: 100nF, PCM_JLCPCB:C_0402, F.Cu at (170.6, 106.5)
- added C77: 100nF, PCM_JLCPCB:C_0402, F.Cu at (170.9, 101.9)
- added C78: 220nF, PCM_JLCPCB:C_0402, F.Cu at (146.4, 104.0)
- added REF**: AMASS_XT30U-F_1x02_P5.0mm_Vertical, Connector_AMASS:AMASS_XT30U-F_1x02_P5.0mm_Vertical, F.Cu at (121.9, 110.8)
- C14, C15: value 220nF -> 100nF
- C23, C24, C25, C26: footprint PCM_JLCPCB:C_0805 -> PCM_JLCPCB:C_0402
- L1: value 4.7uH -> 1uH
- R6: footprint PCM_JLCPCB:R_0402 -> PCM_JLCPCB:R_0603
- TP1, TP10, TP11, TP12, TP13, TP14, TP15, TP16, TP2, TP3, TP4, TP5, TP6, TP7, TP8, TP9, U7, U8: moved to B.Cu
- moved C19 186.8 mm to (250.8, 24.4)
- moved C20 186.8 mm to (258.8, 25.1)
- moved C21 186.8 mm to (250.8, 26.3)
- moved C22 186.8 mm to (250.8, 28.1)
- moved R14 186.8 mm to (254.4, 25.0)
- moved R15 186.8 mm to (254.4, 27.9)
- moved R16 186.8 mm to (254.4, 30.9)
- moved R17 186.8 mm to (250.8, 30.0)
- moved R18 186.8 mm to (250.8, 31.9)
- moved R19 186.8 mm to (258.4, 27.7)
- moved U2 163.1 mm to (173.1, 117.9), turned to 180 degrees
- moved C6 156.5 mm to (173.8, 87.9)
- moved C5 155.6 mm to (167.6, 113.3), turned to 90 degrees
- moved D8 151.9 mm to (153.2, 115.0), turned to -90 degrees
- moved C7 151.6 mm to (169.5, 82.8), turned to 90 degrees
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Connections:
- C23 pad 1: /Power/Battery/VC4 -> /Power/Battery/VC3
- C23 pad 2: /Power/Battery/VC3 -> /Power/Battery/VC2
- C24 pad 1: /Power/Battery/VC3 -> /Power/Battery/VC2
- C24 pad 2: /Power/Battery/VC2 -> /Power/Battery/VC1
- C25 pad 1: /Power/Battery/VC2 -> /Power/Battery/VC1
- C25 pad 2: /Power/Battery/VC1 -> /Power/Battery/VC0
- C26 pad 1: /Power/Battery/VC1 -> /Power/Battery/VC0
- C26 pad 2: /Power/Battery/VC0 -> VSS
- C34 pad 1: /Power/Battery/REG1 -> /MCU_REG
- C36 pad 1: /MCU_REG -> Net-(Q1-C)
- C5 pad 1: +3.3V -> /MCU_REG
- D4 pad 1: Net-(U8--) -> Net-(U8-+)
- F1 pad 1: Net-(U8--) -> Net-(U8-+)
- Q1 pad 3: /MCU_REG -> Net-(Q1-C)
- R31 pad 1: /Power/Battery/RST_SHUT -> /RST_SHUT
- R35 pad 1: /MCU_REG -> Net-(Q1-C)
- TP8 pad 1: /Power/Battery/REG1 -> /MCU_REG
- TP9 pad 1: unconnected-(TP9-Pad1) -> Net-(Q1-E)
- U3 pad 8: +3.3V -> /MCU_REG
- U6 pad 11: /BMSINT -> /SO
- U6 pad 12: /KILL -> /CAN_CS
- U6 pad 13: unconnected-(U6-GPIO10-Pad13) -> /SCK
- U6 pad 14: unconnected-(U6-GPIO11-Pad14) -> /CANINT
- U6 pad 18: /CANRESET -> unconnected-(U6-GPIO15-Pad18)
- U6 pad 27: /CAN_CS -> /SDA1
- U6 pad 28: unconnected-(U6-GPIO17-Pad28) -> /SCL1
- U6 pad 29: /SI -> /BMSINT
- U6 pad 30: /SO -> /KILL
- U6 pad 31: unconnected-(U6-GPIO20-Pad31) -> /RST_SHUT
- U6 pad 32: /SCK -> /CHGINT
- U6 pad 34: /CANINT -> unconnected-(U6-GPIO22-Pad34)
- U6 pad 9: /CHGINT -> /SI
- U8 pad 1: Net-(U8--) -> VSS
- U8 pad 2: VSS -> Net-(U8-+)
- U9 pad 33: /Power/Battery/RST_SHUT -> /RST_SHUT
- U9 pad 35: /Power/Battery/REG1 -> /MCU_REG
Routing:
- net /MCU_REG: track 0.00 -> 80.0 mm, vias 0 -> 5
- net GND: track 0.00 -> 77.6 mm, vias 0 -> 49
- net /SDA1: track 0.00 -> 53.5 mm, vias 0 -> 2
- net /SCL1: track 0.00 -> 53.2 mm, vias 0 -> 2
- net /CHGINT: track 0.00 -> 44.6 mm, vias 0 -> 2
- net VSS: track 0.00 -> 41.5 mm, vias 0 -> 21
- net /RST_SHUT: track 0.00 -> 30.5 mm, vias 0 -> 3
- net /Power/Battery/VC4: track 0.00 -> 25.5 mm
- net /KILL: track 0.00 -> 23.5 mm, vias 0 -> 2
- net /BMSINT: track 0.00 -> 19.7 mm
- net /QSPI_SS: track 0.00 -> 15.0 mm
- net /SI: track 0.00 -> 14.7 mm, vias 0 -> 2
- net /CAN_CS: track 0.00 -> 14.5 mm, vias 0 -> 2
- net /SO: track 0.00 -> 13.7 mm
- net Net-(Q2-G): track 0.00 -> 13.1 mm, vias 0 -> 3
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- added copper zone on F.Cu, net /MCU_REG
- added copper zone on F.Cu, net /Power/Battery/CD
- added copper zone on F.Cu, net /Power/Battery/PACK+
- added copper zone on F.Cu, net /Power/Battery/VBAT
- added copper zone on F.Cu, net /Power/Charger/VIN
- added copper zone on F.Cu, net /USB_REG
- added copper zone on F.Cu, net /VSYS
- added copper zone on In1.Cu, net GND
- added copper zone on In2.Cu, net GND
- added copper zone on F.Cu, net Net-(U10-SW1)
- added copper zone on F.Cu, net Net-(U10-SW2)
- added copper zone on F.Cu, net VSS
- added copper zone on In1.Cu, net VSS
- added copper zone on In2.Cu, net VSS
- removed copper zone on B.Cu, net GND
- removed copper zone on F.Cu, net GND
Other:
- copper layers 2 -> 4
- board text added: "${REFERENCE}"
- board text added: "CHARGER ENTRY POINT"
- board text added: "CHECK ANALOG INTEGRITY"
- board text added: "FIX THIS SHIT"
- board text added: "MCU REG"
- board text added: "SPACE FOR VBAT"
- board text added: "USB TIE"
- board text added: "VIA STITCH VSS"
- board text added: "VIA TO CD"

Commit message: Footprint routing completed
Parts:
- removed J3: Conn_01x02, Connector_PinHeader_2.54mm:PinHeader_1x02_P2.54mm_Vertical
- removed TP20: RH-5015, 4in-power:SMD_RH-5015
- removed U16: SX1308, 4in-power:SOT-23-6_L2.9-W1.6-P0.95-LS2.8-BL
- added C27: 1uF, PCM_JLCPCB:C_0805, F.Cu at (168.7, 82.9)
- added C79: 4.7uF, PCM_JLCPCB:C_1206, F.Cu at (160.8, 73.3)
- added C80: 4.7uF, PCM_JLCPCB:C_1206, F.Cu at (158.5, 73.3)
- added C81: 100nF, PCM_JLCPCB:C_0402, F.Cu at (162.4, 71.7)
- added L2: 2.7uH, 4in-power:IND-SMD_L7.5-W7.5_XAL7030, F.Cu at (171.1, 78.7)
- added R53: 47kΩ, PCM_JLCPCB:R_0402, F.Cu at (167.5, 86.6)
- added R54: 2kΩ, PCM_JLCPCB:R_0402, F.Cu at (174.2, 89.5)
- added R55: 47Ω, PCM_JLCPCB:R_0402, F.Cu at (175.5, 90.1)
- added R56: 10kΩ, PCM_JLCPCB:R_0402, F.Cu at (174.7, 83.9)
- added REF**: AMASS_XT30U-F_1x02_P5.0mm_Vertical, Connector_AMASS:AMASS_XT30U-F_1x02_P5.0mm_Vertical, F.Cu at (155.8, 88.6)
- added U17: 2P SMD 2.54P Jumper, 4in-power:HDR-SMD_2P-P2.54-V-M-S4.8_DZ254S-11-02-50, F.Cu at (157.7, 103.5)
- C70: value 10uF -> 1uF
- C71: value 10uF -> 330pF; footprint PCM_JLCPCB:C_0805 -> PCM_JLCPCB:C_0603
- C72: value 10uF -> 8.2nF; footprint PCM_JLCPCB:C_0805 -> PCM_JLCPCB:C_0603
- C73: value 10uF -> 10nF; footprint PCM_JLCPCB:C_0805 -> PCM_JLCPCB:C_0402
- C74: value 10uF -> 100nF; footprint PCM_JLCPCB:C_0805 -> PCM_JLCPCB:C_0402
- C75: value 10uF -> 1uF; footprint PCM_JLCPCB:C_0805 -> PCM_JLCPCB:C_0603
- D16: value SSL54 -> SS54
- R49: value 1kΩ -> 470Ω; footprint PCM_JLCPCB:R_0402 -> PCM_JLCPCB:R_0603
- R50: value 39kΩ -> 470Ω; footprint PCM_JLCPCB:R_0402 -> PCM_JLCPCB:R_0603
- R51: value 330kΩ -> 9.1kΩ; footprint PCM_JLCPCB:R_0805 -> PCM_JLCPCB:R_0603
- R52: value 100kΩ -> 5.1Ω; footprint PCM_JLCPCB:R_0805 -> PCM_JLCPCB:R_0603
- TP17, TP18, TP19: moved to B.Cu
- U15: value 6.8uH -> LM5157RTER; footprint 4in-power:IND-SMD_L5.4-W5.2_SLO0530H6R8MTT -> 4in-power:WQFN-16_L3.0-W3.0-P0.50-TL-EP1.7
- moved C64 145.9 mm to (127.4, 75.0), turned to 90 degrees
- moved C65 144.8 mm to (128.2, 75.0), turned to 90 degrees
- moved D15 144.5 mm to (132.7, 71.5), turned to 180 degrees
- moved C66 143.8 mm to (129.8, 79.9)
- moved R47 142.7 mm to (126.0, 76.8), turned to -90 degrees
- moved D14 141.4 mm to (146.8, 79.2), turned to 180 degrees
- moved C58 140.9 mm to (141.9, 82.9), turned to 90 degrees
- moved R48 140.7 mm to (127.9, 78.8), turned to -90 degrees
- moved C68 139.9 mm to (138.4, 79.0), turned to -90 degrees
- moved C67 139.6 mm to (132.7, 73.8)
- moved C59 139.4 mm to (142.7, 82.9), turned to 90 degrees
- moved C60 139.3 mm to (144.2, 87.8)
- moved R45 139.0 mm to (140.4, 84.8), turned to -90 degrees
- moved U13 138.6 mm to (132.5, 76.9), turned to -90 degrees
- moved C62 136.9 mm to (147.0, 75.1), turned to -90 degrees
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Connections:
- C68 pad 1: /Power/StepDown3.3V/+5V -> +3.3V
- C69 pad 1: /Power/StepDown3.3V/+5V -> +3.3V
- C70 pad 1: +24V -> /VSYS
- C71 pad 1: +24V -> GND
- C71 pad 2: GND -> Net-(U15-COMP)
- C72 pad 1: +24V -> Net-(U15-COMP)
- C72 pad 2: GND -> Net-(C72-Pad2)
- C73 pad 1: /VSYS -> GND
- C73 pad 2: GND -> Net-(U15-SS)
- C75 pad 1: /VSYS -> Net-(C75-Pad1)
- D16 pad 2: Net-(U16-SW) -> Net-(D16-Pad2)
- J2 pad A1: unconnected-(J2-CANH-PadA1) -> /CANP
- J2 pad A3: unconnected-(J2-CANN-PadA3) -> /CANN
- R17 pad 1: /Power/StepDown3.3V/+5V -> +3.3V
- R49 pad 1: +24V -> Net-(R49-Pad1)
- R49 pad 2: Net-(U16-FB) -> Net-(C72-Pad2)
- R50 pad 1: Net-(U16-FB) -> GND
- R50 pad 2: GND -> Net-(R49-Pad1)
- R51 pad 1: /VSYS -> Net-(U15-RT)
- R51 pad 2: /EN_24V -> GND
- R52 pad 1: /EN_24V -> Net-(U15-VCC)
- R52 pad 2: GND -> Net-(C75-Pad1)
- REF** pad 1: (no net) -> GND
- REF** pad 2: (no net) -> /Power/Charger/VIN
- U14 pad 2: /Power/StepDown3.3V/+5V -> +3.3V
- U15 pad 1: Net-(U16-SW) -> GND
- U15 pad 2: /VSYS -> Net-(U15-VCC)
- U6 pad 15: unconnected-(U6-GPIO12-Pad15) -> CANSTBY
- U6 pad 16: unconnected-(U6-GPIO13-Pad16) -> /EN_24V
- U6 pad 17: unconnected-(U6-GPIO14-Pad17) -> /EN_3.3V
- U6 pad 18: unconnected-(U6-GPIO15-Pad18) -> /EN_5V
- U6 pad 38: CANSTBY -> unconnected-(U6-GPIO26_ADC0-Pad38)
- U6 pad 4: /SDA1 -> unconnected-(U6-GPIO2-Pad4)
- U6 pad 5: /SCL1 -> unconnected-(U6-GPIO3-Pad5)
- U6 pad 6: /EN_3.3V -> unconnected-(U6-GPIO4-Pad6)
- U6 pad 7: /EN_5V -> unconnected-(U6-GPIO5-Pad7)
- U6 pad 8: /EN_24V -> unconnected-(U6-GPIO6-Pad8)
Routing:
- net +3.3V: track 3.21 -> 84.4 mm, vias 0 -> 14
- net /CANP: track 0.00 -> 59.8 mm, vias 0 -> 4
- net /CANN: track 0.00 -> 59.5 mm, vias 0 -> 4
- net GND: track 77.6 -> 136.5 mm, vias 49 -> 114
- net /EN_3.3V: track 0.00 -> 54.9 mm, vias 0 -> 4
- net /EN_5V: track 0.00 -> 38.5 mm, vias 0 -> 2
- net +5V: track 1.20 -> 35.6 mm, vias 0 -> 13
- net /EN_24V: track 0.00 -> 32.9 mm, vias 0 -> 5
- net /VSYS: track 1.85 -> 19.0 mm, vias 1 -> 46
- net +1.1V: track 1.61 -> 15.6 mm, vias 0 -> 3
- net CANSTBY: track 0.00 -> 11.6 mm, vias 0 -> 2
- net +24V: track 0.00 -> 11.0 mm
- net /SWCLK: track 0.00 -> 10.8 mm, vias 0 -> 2
- net /SWD: track 0.00 -> 9.32 mm, vias 0 -> 2
- net Net-(U15-FB): track 0.00 -> 8.72 mm, vias 0 -> 2
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- added copper zone on F.Cu, net +24V
- added copper zone on B.Cu, net +3.3V
- added copper zone on F.Cu, net +3.3V
- added copper zone on B.Cu, net +5V
- added copper zone on F.Cu, net +5V
- added copper zone on F.Cu, net /Power/StepDown3.3V/SW
- added copper zone on F.Cu, net /Power/StepDown5V/SW
- added copper zone on B.Cu, net /VSYS
- added copper zone on B.Cu, net GND
- added copper zone on F.Cu, net GND
- added copper zone on F.Cu, net Net-(D16-Pad2)
Other:
- board text added: "BOOT"
- board text removed: "${REFERENCE}"
- board text removed: "DO LAYOUT FOR THESE BUCKS. 4Layers. Make as compact as possible"
- board text removed: "FIX THIS SHIT"
